File: PCB/agricoltura-vine/Power.sch (KiCad schematic (older format))
At the start: 0 parts

Commit message: Power Supplies
designed power supplies for 3.3v and 5V as well as 24VAC input
Parts:
- added C?: C0805C104M5RACTU, AVR-KiCAD-Lib-Capacitors:C0805, symbol AVR-KiCAD-Lib-Capacitors:C0805C104M5RACTU
- added C?: GRM21BD70J226ME44L, growbox-KiCAD-Capacitors:C0805, symbol AVR-KiCAD-Lib-Capacitors:GRM21BD70J226ME44L
- added C?: CGA3E2X7R1H104K080AA, AVR-KiCAD-Lib-Capacitors:C0603, symbol AVR-KiCAD-Lib-Capacitors:CGA3E2X7R1H104K080AA
- added C?: GRM31CR71H475KA12L, growbox-KiCAD-Capacitors:C1206, symbol AVR-KiCAD-Lib-Capacitors:GRM31CR71H475KA12L
- added C?: GRM32EC72A106KE05L, AVR-KiCAD-Lib-Capacitors:C1210, symbol AVR-KiCAD-Lib-Capacitors:GRM32EC72A106KE05L
- added C? (x2): C2012X7R2A104K125AA, AVR-KiCAD-Lib-Capacitors:C0805, symbol AVR-KiCAD-Lib-Capacitors:C2012X7R2A104K125AA
- added C?: C3216X5R1V156M160AC, AVR-KiCAD-Lib-Capacitors:C1206, symbol AVR-KiCAD-Lib-Capacitors:C3216X5R1V156M160AC
- added D?: ABS210-13, AVR-KiCAD-Lib-Diodes:ABS210-13, symbol AVR-KiCAD-Lib-Diodes:ABS210-13
- added D?: SMDJ15CA, AVR-KiCAD-Lib-Diodes:SMDJ15CA, symbol AVR-KiCAD-Lib-Diodes:SMDJ15CA
- added L?: SDR0403-120ML, AVR-KiCAD-Lib-Inductors:SDR0403-120ML, symbol AVR-KiCAD-Lib-Inductors:SDR0403-120ML
- added L?: SDR0604-180YL, AVR-KiCAD-Lib-Inductors:INDP5858X480N, symbol AVR-KiCAD-Lib-Inductors:SDR0604-180YL
- added R? (x2): RC0402FR-0722K1L, AVR-KiCAD-Lib-Resistors:R0402, symbol AVR-KiCAD-Lib-Resistors:RC0402FR-0722K1L
- added R?: RC0402FR-07412KL, AVR-KiCAD-Lib-Resistors:R0402, symbol AVR-KiCAD-Lib-Resistors:RC0402FR-07412KL
- added R?: RC0402FR-0751KL, AVR-KiCAD-Lib-Resistors:R0402, symbol AVR-KiCAD-Lib-Resistors:RC0402FR-0751KL
- added R?: RC0402FR-07200KL, AVR-KiCAD-Lib-Resistors:R0402, symbol AVR-KiCAD-Lib-Resistors:RC0402FR-07200KL
- added R?: RC0402FR-07750KL, AVR-KiCAD-Lib-Resistors:R0402, symbol AVR-KiCAD-Lib-Resistors:RC0402FR-07750KL
- added R?: CRCW0402294KFKED, AVR-KiCAD-Lib-Resistors:R0402, symbol AVR-KiCAD-Lib-Resistors:CRCW0402294KFKED
- added R?: RC0402FR-0788K7L, AVR-KiCAD-Lib-Resistors:R0402, symbol AVR-KiCAD-Lib-Resistors:RC0402FR-0788K7L
- added T?: 1755736, growbox-KiCAD-Connectors:PhoenixContact_MSTBVA-G_02x5.08mm_Vertical, symbol AVR-KiCAD-Lib-Connectors:1755736
- added U? (x2): TPS560430XDBVR, growbox-KiCAD-ICs:SOT-23-6_Handsoldering, symbol AVR-KiCAD-Lib-ICs:TPS560430XDBVR
Connections:
- net labels added: +24V, +3V3, +5V, GND
- wire segments 0 -> 51
