File: PCB/agricoltura-vine/I2C_Interfaces.sch (KiCad schematic (older format))
At the start: 36 parts, among them T10 BM04B-SRSS-TB(LF)(SN), T11 BM04B-SRSS-TB(LF)(SN), T12 BM04B-SRSS-TB(LF)(SN), T13 BM04B-SRSS-TB(LF)(SN), T14 BM04B-SRSS-TB(LF)(SN), T15 BM04B-SRSS-TB(LF)(SN), T8 BM04B-SRSS-TB(LF)(SN), T9 BM04B-SRSS-TB(LF)(SN), U3 TCA9548APWR

Commit message: Board tweaks
TVS diodes added, board needs routing, a lot of board has been tweaked, more to come.
Parts:
- gave numbers to parts that had none: 9
Changed lines of the file:
@@
 	4200 4500 4050 4500
 $Comp
-L AVR-KiCAD-Lib-Diodes:PESD3V3L2BT,215 D?
+L AVR-KiCAD-Lib-Diodes:PESD3V3L2BT,215 D9
 U 1 1 5F2FDE20
 P 3950 4900
-F 0 "D?" V 3750 5150 50  0000 L CNN
+F 0 "D9" V 3750 5150 50  0000 L CNN
 F 1 "PESD3V3L2BT,215" H 4000 5100 50  0001 C CNN
 F 2 "AVR-KiCAD-Lib-Diodes:SOT-23" H 3850 4900 50  0001 C CNN
@@
 $EndComp
 $Comp
-L AVR-KiCAD-Lib-Diodes:PESD3V3L2BT,215 D?
+L AVR-KiCAD-Lib-Diodes:PESD3V3L2BT,215 D10
 U 1 1 5F301A3E
 P 4650 4900
-F 0 "D?" V 4450 5150 50  0000 L CNN
+F 0 "D10" V 4450 5150 50  0000 L CNN
 F 1 "PESD3V3L2BT,215" H 4700 5100 50  0001 C CNN
 F 2 "AVR-KiCAD-Lib-Diodes:SOT-23" H 4550 4900 50  0001 C CNN
@@
 	4750 2400 3250 2400
 $Comp
-L AVR-KiCAD-Lib-Diodes:PESD3V3L2BT,215 D?
+L AVR-KiCAD-Lib-Diodes:PESD3V3L2BT,215 D11
 U 1 1 5F31E3E5
 P 5300 4900
-F 0 "D?" V 5100 5150 50  0000 L CNN
+F 0 "D11" V 5100 5150 50  0000 L CNN
 F 1 "PESD3V3L2BT,215" H 5350 5100 50  0001 C CNN
 F 2 "AVR-KiCAD-Lib-Diodes:SOT-23" H 5200 4900 50  0001 C CNN
@@
 	7150 3500 7150 4650
 $Comp
-L AVR-KiCAD-Lib-Diodes:PESD3V3L2BT,215 D?
+L AVR-KiCAD-Lib-Diodes:PESD3V3L2BT,215 D12
 U 1 1 5F34DA9D
 P 5950 4900
-F 0 "D?" V 5750 5150 50  0000 L CNN
+F 0 "D12" V 5750 5150 50  0000 L CNN
 F 1 "PESD3V3L2BT,215" H 6000 5100 50  0001 C CNN
 F 2 "AVR-KiCAD-Lib-Diodes:SOT-23" H 5850 4900 50  0001 C CNN
@@
 $EndComp
 $Comp
-L AVR-KiCAD-Lib-Diodes:PESD3V3L2BT,215 D?
+L AVR-KiCAD-Lib-Diodes:PESD3V3L2BT,215 D13
 U 1 1 5F34E9EA
 P 6600 4900
-F 0 "D?" V 6400 5150 50  0000 L CNN
+F 0 "D13" V 6400 5150 50  0000 L CNN
 F 1 "PESD3V3L2BT,215" H 6650 5100 50  0001 C CNN
 F 2 "AVR-KiCAD-Lib-Diodes:SOT-23" H 6500 4900 50  0001 C CNN
@@
 $EndComp
 $Comp
-L AVR-KiCAD-Lib-Diodes:PESD3V3L2BT,215 D?
+L AVR-KiCAD-Lib-Diodes:PESD3V3L2BT,215 D14
 U 1 1 5F34F4A9
 P 7250 4900
-F 0 "D?" V 7050 5150 50  0000 L CNN
+F 0 "D14" V 7050 5150 50  0000 L CNN
 F 1 "PESD3V3L2BT,215" H 7300 5100 50  0001 C CNN
 F 2 "AVR-KiCAD-Lib-Diodes:SOT-23" H 7150 4900 50  0001 C CNN
@@
 $EndComp
 $Comp
-L AVR-KiCAD-Lib-Diodes:PESD3V3L2BT,215 D?
+L AVR-KiCAD-Lib-Diodes:PESD3V3L2BT,215 D15
 U 1 1 5F350A3C
 P 7550 5500
-F 0 "D?" V 7350 5750 50  0000 L CNN
+F 0 "D15" V 7350 5750 50  0000 L CNN
 F 1 "PESD3V3L2BT,215" H 7600 5700 50  0001 C CNN
 F 2 "AVR-KiCAD-Lib-Diodes:SOT-23" H 7450 5500 50  0001 C CNN
@@
 	7900 3900 3250 3900
 $Comp
-L AVR-KiCAD-Lib-Diodes:PESD3V3L2BT,215 D?
+L AVR-KiCAD-Lib-Diodes:PESD3V3L2BT,215 D16
 U 1 1 5F384AF8
 P 8400 6100
-F 0 "D?" V 8200 6350 50  0000 L CNN
+F 0 "D16" V 8200 6350 50  0000 L CNN
 F 1 "PESD3V3L2BT,215" H 8450 6300 50  0001 C CNN
 F 2 "AVR-KiCAD-Lib-Diodes:SOT-23" H 8300 6100 50  0001 C CNN
@@
 	8500 5050 8850 5050
 $Comp
-L AVR-KiCAD-Lib-Diodes:PESD3V3L2BT,215 D?
+L AVR-KiCAD-Lib-Diodes:PESD3V3L2BT,215 D17
 U 1 1 5F396FBB
 P 9200 6100
-F 0 "D?" V 9000 6350 50  0000 L CNN
+F 0 "D17" V 9000 6350 50  0000 L CNN
 F 1 "PESD3V3L2BT,215" H 9250 6300 50  0001 C CNN
 F 2 "AVR-KiCAD-Lib-Diodes:SOT-23" H 9100 6100 50  0001 C CNN
@@
 P 3050 5200
 AR Path="/5EE82896/5F3CD023" Ref="#PWR?"  Part="1"
-AR Path="/5EE827B2/5F3CD023" Ref="#PWR?"  Part="1"
-F 0 "#PWR?" H 3050 5050 50  0001 C CNN
+AR Path="/5EE827B2/5F3CD023" Ref="#PWR0139"  Part="1"
+F 0 "#PWR0139" H 3050 5050 50  0001 C CNN
 F 1 "+3V3" H 3065 5373 50  0000 C CNN
 F 2 "" H 3050 5200 50  0001 C CNN

Commit message: TVS Diodes
TVS diodes and pullups added to sensor connectors, implemented in schematic and board.
Parts:
- removed D17: PESD3V3L2BT,215, AVR-KiCAD-Lib-Diodes:SOT-23, symbol AVR-KiCAD-Lib-Diodes:PESD3V3L2BT,215
Connections:
- net QWIIC_SC0: now also D10.1; no longer D10.2
- net QWIIC_SC1: now also D11.1; no longer D11.2
- net QWIIC_SC2: now also D12.1; no longer D12.2
- net QWIIC_SC3: now also D13.1; no longer D13.2
- net QWIIC_SC4: now also D14.1; no longer D14.2
- net QWIIC_SC5: now also D15.1; no longer D15.2
- net QWIIC_SC6: now also D16.1; no longer D16.2
- net QWIIC_SC7: now also D9.1; no longer D9.2
- net QWIIC_SD0: now also D10.2; no longer D10.1
- net QWIIC_SD1: now also D11.2; no longer D11.1
- net QWIIC_SD2: now also D12.2; no longer D12.1
- net QWIIC_SD3: now also D13.2; no longer D13.1
- net QWIIC_SD4: now also D14.2; no longer D14.1
- net QWIIC_SD5: now also D15.2; no longer D15.1
- net QWIIC_SD6: now also D16.2; no longer D16.1
- net QWIIC_SD7: now also D9.2; no longer D9.1
Changed lines of the file:
@@
 	8100 4400 8100 5650
-Wire Wire Line
-	8100 5650 9100 5650
-Wire Wire Line
-	10600 5750 9300 5750
 Wire Wire Line
 	8000 5750 8000 4500
@@
 	4200 2200 4200 4500
 Connection ~ 4200 4500
-Wire Wire Line
-	4200 4500 4050 4500
-$Comp
-L AVR-KiCAD-Lib-Diodes:PESD3V3L2BT,215 D9
-U 1 1 5F2FDE20
-P 3950 4900
-F 0 "D9" V 3750 5150 50  0000 L CNN
-F 1 "PESD3V3L2BT,215" H 4000 5100 50  0001 C CNN
-F 2 "AVR-KiCAD-Lib-Diodes:SOT-23" H 3850 4900 50  0001 C CNN
-F 3 "https://assets.nexperia.com/documents/data-sheet/PESDXL2BT_SER.pdf" H 3850 5000 50  0001 C CNN
-F 4 "0.45000" H 4050 5150 50  0001 C CNN "Cost QTY: 1"
-F 5 "0.13260" H 4150 5250 50  0001 C CNN "Cost QTY: 1000"
-F 6 "*" H 4250 5350 50  0001 C CNN "Cost QTY: 2500"
-F 7 "*" H 4350 5450 50  0001 C CNN "Cost QTY: 5000"
-F 8 "*" H 4450 5550 50  0001 C CNN "Cost QTY: 10000"
-F 9 "Nexperia USA Inc." H 4550 5650 50  0001 C CNN "MFR"
-F 10 "PESD3V3L2BT,215" H 4650 5750 50  0001 C CNN "MFR#"
-F 11 "Digikey" H 4750 5850 50  0001 C CNN "Vendor"
-F 12 "1727-3826-1-ND" H 4850 5950 50  0001 C CNN "Vendor #"
-F 13 "AVR" H 4950 6050 50  0001 C CNN "Designer"
-F 14 "1.1mm" H 5050 6150 50  0001 C CNN "Height"
-F 15 "6/15/2020" H 6150 7250 50  0001 C CNN "Date Created"
-F 16 "6/15/2020" H 5150 6250 50  0001 C CNN "Date Modified"
-F 17 "Yes" H 5250 6350 50  0001 C CNN "Lead-Free ?"
-F 18 "1" H 5350 6450 50  0001 C CNN "RoHS Levels"
-F 19 "SMT" H 5450 6550 50  0001 C CNN "Mounting"
-F 20 "3" H 5550 6650 50  0001 C CNN "Pin Count #"
-F 21 "Active" H 5650 6750 50  0001 C CNN "Status"
-F 22 "*" H 5750 6850 50  0001 C CNN "Tolerance"
-F 23 "TVS" H 5850 6950 50  0001 C CNN "Type"
-F 24 "*" H 5950 7050 50  0001 C CNN "Voltage"
-F 25 " SOT-23-3" H 6050 7200 50  0001 C CNN "Package"
-F 26 "26V Clamp 15A (8/20µs) Ipp Tvs Diode Surface Mount TO-236AB" H 6350 7500 50  0001 C CNN "Description"
-F 27 "PESD3V3L2BT,215" V 4200 4150 50  0000 L CNN "_Value_"
-F 28 "*" H 6350 7500 50  0001 C CNN "Management_ID"
-	1    3950 4900
-	0    1    1    0
-$EndComp
 $Comp
 L AVR-KiCAD-Lib-Diodes:PESD3V3L2BT,215 D10
@@
 F 25 " SOT-23-3" H 6750 7200 50  0001 C CNN "Package"
 F 26 "26V Clamp 15A (8/20µs) Ipp Tvs Diode Surface Mount TO-236AB" H 7050 7500 50  0001 C CNN "Description"
-F 27 "PESD3V3L2BT,215" V 5050 4200 50  0000 L CNN "_Value_"
+F 27 "PESD3V3L2BT,215" V 5050 4950 50  0000 L CNN "_Value_"
 F 28 "*" H 7050 7500 50  0001 C CNN "Management_ID"
 	1    4650 4900
-	0    1    1    0
+	0    -1   1    0
 $EndComp
 Wire Wire Line
 	4550 2300 4550 4650
-Wire Wire Line
-	3850 4400 3850 4650
-Wire Wire Line
-	4050 4650 4050 4500
-Connection ~ 4050 4500
-Wire Wire Line
-	4050 4500 3250 4500
 Wire Wire Line
 	4750 4650 4750 2400
@@
 F 25 " SOT-23-3" H 7400 7200 50  0001 C CNN "Package"
 F 26 "26V Clamp 15A (8/20µs) Ipp Tvs Diode Surface Mount TO-236AB" H 7700 7500 50  0001 C CNN "Description"
-F 27 "PESD3V3L2BT,215" V 5700 4250 50  0000 L CNN "_Value_"
+F 27 "PESD3V3L2BT,215" V 5700 4800 50  0000 L CNN "_Value_"
 F 28 "*" H 7700 7500 50  0001 C CNN "Management_ID"
 	1    5300 4900
-	0    1    1    0
+	0    -1   1    0
 $EndComp
 Wire Wire Line
@@
 F 25 " SOT-23-3" H 8050 7200 50  0001 C CNN "Package"
 F 26 "26V Clamp 15A (8/20µs) Ipp Tvs Diode Surface Mount TO-236AB" H 8350 7500 50  0001 C CNN "Description"
-F 27 "PESD3V3L2BT,215" V 6350 4400 50  0000 L CNN "_Value_"
+F 27 "PESD3V3L2BT,215" V 6350 4650 50  0000 L CNN "_Value_"
 F 28 "*" H 8350 7500 50  0001 C CNN "Management_ID"
 	1    5950 4900
-	0    1    1    0
+	0    -1   1    0
 $EndComp
 $Comp
@@
 F 28 "*" H 9000 7500 50  0001 C CNN "Management_ID"
 	1    6600 4900
-	0    1    1    0
+	0    -1   1    0
 $EndComp
 $Comp
@@
 F 25 " SOT-23-3" H 9350 7200 50  0001 C CNN "Package"
 F 26 "26V Clamp 15A (8/20µs) Ipp Tvs Diode Surface Mount TO-236AB" H 9650 7500 50  0001 C CNN "Description"
-F 27 "PESD3V3L2BT,215" H 7000 5100 50  0000 L CNN "_Value_"
+F 27 "PESD3V3L2BT,215" H 6900 4650 50  0000 L CNN "_Value_"
 F 28 "*" H 9650 7500 50  0001 C CNN "Management_ID"
 	1    7250 4900
-	0    1    1    0
+	0    -1   1    0
 $EndComp
 $Comp
@@
 F 25 " SOT-23-3" H 9650 7800 50  0001 C CNN "Package"
 F 26 "26V Clamp 15A (8/20µs) Ipp Tvs Diode Surface Mount TO-236AB" H 9950 8100 50  0001 C CNN "Description"
-F 27 "PESD3V3L2BT,215" H 7300 5700 50  0000 L CNN "_Value_"
+F 27 "PESD3V3L2BT,215" H 7150 5300 50  0000 L CNN "_Value_"
 F 28 "*" H 9950 8100 50  0001 C CNN "Management_ID"
 	1    7550 5500
-	-1   0    0    1
+	-1   0    0    -1
 $EndComp
 Wire Wire Line
@@
 F 25 " SOT-23-3" H 10500 8400 50  0001 C CNN "Package"
 F 26 "26V Clamp 15A (8/20µs) Ipp Tvs Diode Surface Mount TO-236AB" H 10800 8700 50  0001 C CNN "Description"
-F 27 "PESD3V3L2BT,215" H 8150 6300 50  0000 L CNN "_Value_"
+F 27 "PESD3V3L2BT,215" H 8100 5900 50  0000 L CNN "_Value_"
 F 28 "*" H 10800 8700 50  0001 C CNN "Management_ID"
 	1    8400 6100
-	0    1    1    0
+	0    -1   1    0
 $EndComp
 Wire Wire Line
@@
 Wire Wire Line
 	8500 5050 8850 5050
-$Comp
-L AVR-KiCAD-Lib-Diodes:PESD3V3L2BT,215 D17
-U 1 1 5F396FBB
-P 9200 6100
-F 0 "D17" V 9000 6350 50  0000 L CNN
-F 1 "PESD3V3L2BT,215" H 9250 6300 50  0001 C CNN
-F 2 "AVR-KiCAD-Lib-Diodes:SOT-23" H 9100 6100 50  0001 C CNN
-F 3 "https://assets.nexperia.com/documents/data-sheet/PESDXL2BT_SER.pdf" H 9100 6200 50  0001 C CNN
-F 4 "0.45000" H 9300 6350 50  0001 C CNN "Cost QTY: 1"
-F 5 "0.13260" H 9400 6450 50  0001 C CNN "Cost QTY: 1000"
-F 6 "*" H 9500 6550 50  0001 C CNN "Cost QTY: 2500"
-F 7 "*" H 9600 6650 50  0001 C CNN "Cost QTY: 5000"
-F 8 "*" H 9700 6750 50  0001 C CNN "Cost QTY: 10000"
-F 9 "Nexperia USA Inc." H 9800 6850 50  0001 C CNN "MFR"
-F 10 "PESD3V3L2BT,215" H 9900 6950 50  0001 C CNN "MFR#"
-F 11 "Digikey" H 10000 7050 50  0001 C CNN "Vendor"
-F 12 "1727-3826-1-ND" H 10100 7150 50  0001 C CNN "Vendor #"
-F 13 "AVR" H 10200 7250 50  0001 C CNN "Designer"
-F 14 "1.1mm" H 10300 7350 50  0001 C CNN "Height"
-F 15 "6/15/2020" H 11400 8450 50  0001 C CNN "Date Created"
-F 16 "6/15/2020" H 10400 7450 50  0001 C CNN "Date Modified"
-F 17 "Yes" H 10500 7550 50  0001 C CNN "Lead-Free ?"
-F 18 "1" H 10600 7650 50  0001 C CNN "RoHS Levels"
-F 19 "SMT" H 10700 7750 50  0001 C CNN "Mounting"
-F 20 "3" H 10800 7850 50  0001 C CNN "Pin Count #"
-F 21 "Active" H 10900 7950 50  0001 C CNN "Status"
-F 22 "*" H 11000 8050 50  0001 C CNN "Tolerance"
-F 23 "TVS" H 11100 8150 50  0001 C CNN "Type"
-F 24 "*" H 11200 8250 50  0001 C CNN "Voltage"
-F 25 " SOT-23-3" H 11300 8400 50  0001 C CNN "Package"
-F 26 "26V Clamp 15A (8/20µs) Ipp Tvs Diode Surface Mount TO-236AB" H 11600 8700 50  0001 C CNN "Description"
-F 27 "PESD3V3L2BT,215" H 8950 6300 50  0000 L CNN "_Value_"
-F 28 "*" H 11600 8700 50  0001 C CNN "Management_ID"
-	1    9200 6100
-	0    1    1    0
-$EndComp
-Wire Wire Line
-	9100 5850 9100 5650
-Connection ~ 9100 5650
-Wire Wire Line
-	9100 5650 10600 5650
-Wire Wire Line
-	9300 5850 9300 5750
-Connection ~ 9300 5750
-Wire Wire Line
-	9300 5750 8000 5750
-Wire Wire Line
-	9200 6400 8400 6400
 Wire Wire Line
 	8400 6400 7250 6400
 Wire Wire Line
 	7250 6400 7250 5500
-Connection ~ 8400 6400
 Connection ~ 7250 5500
 Wire Wire Line
@@
 Wire Wire Line
 	7250 5200 6600 5200
-Connection ~ 3950 5200
-Wire Wire Line
-	3950 5200 3050 5200
 Connection ~ 4650 5200
-Wire Wire Line
-	4650 5200 3950 5200
 Connection ~ 5300 5200
 Wire Wire Line
@@
 Wire Wire Line
 	7350 3600 3250 3600
+Wire Wire Line
+	4050 4500 3250 4500
+Wire Wire Line
+	4200 4500 4050 4500
+Connection ~ 4050 4500
+Wire Wire Line
+	4050 4650 4050 4500
+Wire Wire Line
+	3850 4400 3850 4650
+Connection ~ 3950 5200
+Wire Wire Line
+	3950 5200 3050 5200
+Wire Wire Line
+	4650 5200 3950 5200
+$Comp
+L AVR-KiCAD-Lib-Diodes:PESD3V3L2BT,215 D9
+U 1 1 5F2FDE20
+P 3950 4900
+F 0 "D9" V 3750 5150 50  0000 L CNN
+F 1 "PESD3V3L2BT,215" H 4000 5100 50  0001 C CNN
+F 2 "AVR-KiCAD-Lib-Diodes:SOT-23" H 3850 4900 50  0001 C CNN
+F 3 "https://assets.nexperia.com/documents/data-sheet/PESDXL2BT_SER.pdf" H 3850 5000 50  0001 C CNN
+F 4 "0.45000" H 4050 5150 50  0001 C CNN "Cost QTY: 1"
+F 5 "0.13260" H 4150 5250 50  0001 C CNN "Cost QTY: 1000"
+F 6 "*" H 4250 5350 50  0001 C CNN "Cost QTY: 2500"
+F 7 "*" H 4350 5450 50  0001 C CNN "Cost QTY: 5000"
+F 8 "*" H 4450 5550 50  0001 C CNN "Cost QTY: 10000"
+F 9 "Nexperia USA Inc." H 4550 5650 50  0001 C CNN "MFR"
+F 10 "PESD3V3L2BT,215" H 4650 5750 50  0001 C CNN "MFR#"
+F 11 "Digikey" H 4750 5850 50  0001 C CNN "Vendor"
+F 12 "1727-3826-1-ND" H 4850 5950 50  0001 C CNN "Vendor #"
+F 13 "AVR" H 4950 6050 50  0001 C CNN "Designer"
+F 14 "1.1mm" H 5050 6150 50  0001 C CNN "Height"
+F 15 "6/15/2020" H 6150 7250 50  0001 C CNN "Date Created"
+F 16 "6/15/2020" H 5150 6250 50  0001 C CNN "Date Modified"
+F 17 "Yes" H 5250 6350 50  0001 C CNN "Lead-Free ?"
+F 18 "1" H 5350 6450 50  0001 C CNN "RoHS Levels"
+F 19 "SMT" H 5450 6550 50  0001 C CNN "Mounting"
+F 20 "3" H 5550 6650 50  0001 C CNN "Pin Count #"
+F 21 "Active" H 5650 6750 50  0001 C CNN "Status"
+F 22 "*" H 5750 6850 50  0001 C CNN "Tolerance"
+F 23 "TVS" H 5850 6950 50  0001 C CNN "Type"
+F 24 "*" H 5950 7050 50  0001 C CNN "Voltage"
+F 25 " SOT-23-3" H 6050 7200 50  0001 C CNN "Package"
+F 26 "26V Clamp 15A (8/20µs) Ipp Tvs Diode Surface Mount TO-236AB" H 6350 7500 50  0001 C CNN "Description"
+F 27 "PESD3V3L2BT,215" V 4000 5050 50  0000 L CNN "_Value_"
+F 28 "*" H 6350 7500 50  0001 C CNN "Management_ID"
+	1    3950 4900
+	0    -1   1    0
+$EndComp
+Wire Wire Line
+	8100 5650 10600 5650
+Wire Wire Line
+	8000 5750 10600 5750
 $EndSCHEMATC
